File: ECAD/PCB_Project/MCU.kicad_sch (KiCad schematic)
At the start: 3 parts, among them J401 Conn_01x10, J402 Conn_01x10, J403 Conn_01x02

Commit message: Pushing
COde changes:
MP driver under development
SG90 as well

PCB:
final version, as sent to manufacture

Sims
New sims for report.
Other:
- company: (none) -> Group 9
- title: (none) -> EE318 - Slam Dunk Your Junk
Changed lines of the file:
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@@
 	(generator_version "8.0")
 	(paper "A4")
+	(title_block
+		(title "EE318 - Slam Dunk Your Junk")
+		(date "2024-05-01")
+		(rev "V1")
+		(company "Group 9")
+		(comment 1 "Manufactured Design")
+	)
 	(no_connect
 		(at 109.22 92.71)
@@
 	)
 	(bus_entry
-		(at 46.99 62.23)
+		(at 74.93 101.6)
 		(size 2.54 2.54)
 		(stroke
@@
 	)
 	(bus_entry
-		(at 46.99 59.69)
+		(at 74.93 99.06)
 		(size 2.54 2.54)
 		(stroke
@@
 	)
 	(bus_entry
-		(at 46.99 36.83)
+		(at 74.93 76.2)
 		(size 2.54 2.54)
 		(stroke
@@
 	)
 	(bus_entry
-		(at 46.99 31.75)
+		(at 74.93 71.12)
 		(size 2.54 2.54)
 		(stroke
@@
 	)
 	(bus_entry
-		(at 46.99 39.37)
+		(at 74.93 78.74)
 		(size 2.54 2.54)
 		(stroke
@@
 	)
 	(bus_entry
-		(at 46.99 29.21)
+		(at 74.93 68.58)
 		(size 2.54 2.54)
 		(stroke
@@
 	)
 	(bus_entry
-		(at 46.99 48.26)
+		(at 74.93 87.63)
 		(size 2.54 2.54)
 		(stroke
@@
 	)
 	(bus_entry
-		(at 46.99 34.29)
+		(at 74.93 73.66)
 		(size 2.54 2.54)
 		(stroke
@@
 	)
 	(bus_entry
-		(at 46.99 50.8)
+		(at 74.93 90.17)
 		(size 2.54 2.54)
 		(stroke
@@
 	(wire
 		(pts
-			(xy 44.45 76.2) (xy 49.53 76.2)
+			(xy 72.39 115.57) (xy 77.47 115.57)
 		)
 		(stroke
@@
 	(bus
 		(pts
-			(xy 46.99 46.99) (xy 46.99 48.26)
+			(xy 74.93 86.36) (xy 74.93 87.63)
 		)
 		(stroke
@@
 	(bus
 		(pts
-			(xy 46.99 36.83) (xy 46.99 39.37)
-		)
-		(stroke
-			(width 0)
-			(type default)
-		)
-	)
-	(bus
-		(pts
-			(xy 46.99 58.42) (xy 46.99 59.69)
+			(xy 74.93 76.2) (xy 74.93 78.74)
+		)
+		(stroke
+			(width 0)
+			(type default)
+		)
+	)
+	(bus
+		(pts
+			(xy 74.93 97.79) (xy 74.93 99.06)
 		)
 		(stroke
@@
 	(wire
 		(pts
-			(xy 44.45 83.82) (xy 49.53 83.82)
+			(xy 72.39 123.19) (xy 77.47 123.19)
 		)
 		(stroke
@@
 	(bus
 		(pts
-			(xy 45.72 46.99) (xy 46.99 46.99)
+			(xy 73.66 86.36) (xy 74.93 86.36)
 		)
 		(stroke
@@
 	(bus
 		(pts
-			(xy 46.99 34.29) (xy 46.99 36.83)
-		)
-		(stroke
-			(width 0)
-			(type default)
-		)
-	)
-	(bus
-		(pts
-			(xy 46.99 59.69) (xy 46.99 62.23)
+			(xy 74.93 73.66) (xy 74.93 76.2)
+		)
+		(stroke
+			(width 0)
+			(type default)
+		)
+	)
+	(bus
+		(pts
+			(xy 74.93 99.06) (xy 74.93 101.6)
 		)
 		(stroke
@@
 	(bus
 		(pts
-			(xy 45.72 26.67) (xy 46.99 26.67)
-		)
-		(stroke
-			(width 0)
-			(type default)
-		)
-	)
-	(bus
-		(pts
-			(xy 46.99 26.67) (xy 46.99 29.21)
+			(xy 73.66 66.04) (xy 74.93 66.04)
+		)
+		(stroke
+			(width 0)
+			(type default)
+		)
+	)
+	(bus
+		(pts
+			(xy 74.93 66.04) (xy 74.93 68.58)
 		)
 		(stroke
@@
 	(bus
 		(pts
-			(xy 45.72 58.42) (xy 46.99 58.42)
-		)
-		(stroke
-			(width 0)
-			(type default)
-		)
-	)
-	(wire
-		(pts
-			(xy 44.45 80.01) (xy 49.53 80.01)
+			(xy 73.66 97.79) (xy 74.93 97.79)
+		)
+		(stroke
+			(width 0)
+			(type default)
+		)
+	)
+	(wire
+		(pts
+			(xy 72.39 119.38) (xy 77.47 119.38)
 		)
 		(stroke
@@
 	(bus
 		(pts
-			(xy 46.99 48.26) (xy 46.99 50.8)
-		)
-		(stroke
-			(width 0)
-			(type default)
-		)
-	)
-	(bus
-		(pts
-			(xy 46.99 29.21) (xy 46.99 31.75)
+			(xy 74.93 87.63) (xy 74.93 90.17)
+		)
+		(stroke
+			(width 0)
+			(type default)
+		)
+	)
+	(bus
+		(pts
+			(xy 74.93 68.58) (xy 74.93 71.12)
 		)
 		(stroke
@@
 	(bus
 		(pts
-			(xy 46.99 31.75) (xy 46.99 34.29)
+			(xy 74.93 71.12) (xy 74.93 73.66)
 		)
 		(stroke
@@
 	)
 	(rectangle
-		(start 12.7 17.78)
-		(end 76.2 95.25)
+		(start 40.64 57.15)
+		(end 104.14 134.62)
 		(stroke
 			(width 0)
@@
 	(text_box "Offsheet connections"
 		(exclude_from_sim no)
-		(at 13.97 19.05 0)
+		(at 41.91 58.42 0)
 		(size 24.13 3.81)
 		(stroke
@@
 	)
 	(label "DISPLAY.NCS"
-		(at 49.53 31.75 0)
+		(at 77.47 71.12 0)
 		(fields_autoplaced yes)
 		(effects
@@
 	)
 	(label "Driver.STEP"
-		(at 49.53 62.23 0)
+		(at 77.47 101.6 0)
 		(fields_autoplaced yes)
 		(effects
@@
 	)
 	(label "DISPLAY.SDI"
-		(at 49.53 34.29 0)
+		(at 77.47 73.66 0)
 		(fields_autoplaced yes)
 		(effects
@@
 	)
 	(label "Driver.DIR"
-		(at 49.53 64.77 0)
+		(at 77.47 104.14 0)
 		(fields_autoplaced yes)
 		(effects
@@
 	)
 	(label "DISPLAY.NRST"
-		(at 49.53 39.37 0)
+		(at 77.47 78.74 0)
 		(fields_autoplaced yes)
 		(effects
@@
 	)
 	(label "Ultrasonic.Trigg"
-		(at 49.53 50.8 0)
+		(at 77.47 90.17 0)
 		(fields_autoplaced yes)
 		(effects
@@
 	)
 	(label "Ind_Analog"
-		(at 49.53 80.01 0)
+		(at 77.47 119.38 0)
 		(fields_autoplaced yes)
 		(effects
@@
 	)
 	(label "LDR_Analog"
-		(at 49.53 76.2 0)
+		(at 77.47 115.57 0)
 		(fields_autoplaced yes)
 		(effects
@@
 	)
 	(label "DISPLAY.SCL"
-		(at 49.53 36.83 0)
+		(at 77.47 76.2 0)
 		(fields_autoplaced yes)
 		(effects
@@
 	)
 	(label "SG90_PWM"
-		(at 49.53 83.82 0)
+		(at 77.47 123.19 0)
 		(fields_autoplaced yes)
 		(effects
@@
 	)
 	(label "Ultrasonic.Echo"
-		(at 49.53 53.34 0)
+		(at 77.47 92.71 0)
 		(fields_autoplaced yes)
 		(effects
@@
 	)
 	(label "DISPLAY.A0"
-		(at 49.53 41.91 0)
+		(at 77.47 81.28 0)
 		(fields_autoplaced yes)
 		(effects
@@
 	(hierarchical_label "Ultrasonic{Trigg,Echo}"
 		(shape bidirectional)
-		(at 45.72 46.99 180)
+		(at 73.66 86.36 180)
 		(fields_autoplaced yes)
 		(effects
@@
 	(hierarchical_label "DISPLAY{NCS,SDI,SCL,NRST,A0}"
 		(shape bidirectional)
-		(at 45.72 26.67 180)
+		(at 73.66 66.04 180)
 		(fields_autoplaced yes)
 		(effects
@@
 	(hierarchical_label "Driver{STEP,DIR}"
 		(shape output)
-		(at 45.72 58.42 180)
+		(at 73.66 97.79 180)
 		(fields_autoplaced yes)
 		(effects
@@
 	(hierarchical_label "Ind_3v3"
 		(shape input)
-		(at 44.45 80.01 180)
+		(at 72.39 119.38 180)
 		(fields_autoplaced yes)
 		(effects
@@
 	(hierarchical_label "LDR"
 		(shape input)
-		(at 44.45 76.2 180)
+		(at 72.39 115.57 180)
 		(fields_autoplaced yes)
 		(effects
@@
 	(hierarchical_label "SG90_PWM"
 		(shape output)
-		(at 44.45 83.82 180)
-		(fields_autoplaced yes)
-		(effects
+		(at 72.39 123.19 180)
+		(fields_autoplaced yes)
+		(effects
